Commit message: June20: Test00 and Test01 working!

File: ArmModels/urdfs/P4/P4_Contra-Angle_left.urdf (robot description, URDF)
Before this commit: robot P4.SLDASM, 9 links, 8 joints
Links:
- removed link Weight
Joints:
- removed joint Sensor Flange

File: ArmModels/urdfs/P4/P4_Contra-Angle_right.urdf (robot description, URDF)
Before this commit: robot P4.SLDASM, 9 links, 8 joints
Links:
- link Weight: mass 10.0 -> 10
