Commit message: June26: Modified LOTS of codes - extremely good PD control (tuned parameters), following trajectory, shifted away from fourier trajectory (but need to go back since the other trajectories, although stable are not exciting enough)

File: ArmModels/urdfs/P4/P4_Contra-Angle_right.urdf (robot description, URDF)
Before this commit: robot P4.SLDASM, 9 links, 8 joints
Links:
- link Weight: mass 10 -> 1

Commit message: July03: perfect identification

File: ArmModels/urdfs/P4/P4_Contra-Angle_right.urdf (robot description, URDF)
Before this commit: robot P4.SLDASM, 9 links, 8 joints
Links:
- link Base: geometry collision mesh filename=/home/robot/dev/dyn/ArmModels/meshes/P4/Base_collision.STL; visual mesh filename=/home/robot/dev/dyn/ArmModels/meshes/P4/Base.STL
- link End_Effector: geometry collision capsule length=0.054 radius=0.009; collision mesh filename=/home/robot/dev/dyn/ArmModels/meshes/P4/End_Effector_Contra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
- link Link_0: geometry collision mesh filename=/home/robot/dev/dyn/ArmModels/meshes/P4/Link_0_a_collision.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; collision mesh filename=/home/robot/dev/dyn/ArmModels/meshes/P4/Link_0_b_collision.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
- link Link_1: geometry collision mesh filename=/home/robot/dev/dyn/ArmModels/meshes/P4/Link_1_collision.STL; visual mesh filename=/home/robot/dev/dyn/ArmModels/meshes/P4/Link_1.STL
- link Link_2: geometry collision capsule length=0.09 radius=0.066; collision capsule length=0.125356 radius=0.066
- link Link_3: geometry collision mesh filename=/home/robot/dev/dyn/ArmModels/meshes/P4/Link_3_a_collision.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; collision mesh filename=/home/robot/dev/dyn/ArmModels/meshes/P4/Link_3_b_collision.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
- link Link_4: geometry collision mesh filename=/home/robot/dev/dyn/ArmModels/meshes/P4/Link_4_collision.STL; visual mesh filename=/home/robot/dev/dyn/ArmModels/meshes/P4/Link_4.STL
- link Link_5: geometry collision mesh filename=/home/robot/dev/dyn/ArmModels/meshes/P4/Link_5_collision.STL; visual mesh filename=/home/robot/dev/dyn/ArmModels/meshes/P4/Link_5.STL
Joints:
- joint Joint_0: limit lower=0 upper=0 effort=0 velocity=0 -> lower=-6.28 upper=6.28 effort=10000 velocity=2.5
- joint Joint_1: limit lower=0 upper=0 effort=0 velocity=0 -> lower=-6.28 upper=6.28 effort=10000 velocity=2.5
- joint Joint_2: limit lower=0 upper=0 effort=0 velocity=0 -> lower=-6.28 upper=6.28 effort=10000 velocity=2.5
- joint Joint_3: limit lower=0 upper=0 effort=0 velocity=0 -> lower=-6.28 upper=6.28 effort=10000 velocity=2.5
- joint Joint_4: limit lower=0 upper=0 effort=0 velocity=0 -> lower=-6.28 upper=6.28 effort=10000 velocity=2.5
- joint Joint_5: limit lower=0 upper=0 effort=0 velocity=0 -> lower=-6.28 upper=6.28 effort=10000 velocity=2.5
- joint Joint_6: limit lower=0 upper=0 effort=0 velocity=0 -> lower=-6.28 upper=6.28 effort=10000 velocity=2.5
