Commit message: July17: added base parameter identification and also new PD base params test! -- use this from now on

File: 3DOF/urdf/3DOF Yomi Assembly_Anush.urdf (robot description, URDF)
Before this commit: robot 3DOF, 6 links, 5 joints
Links:
- link End_effector: mass 19.1894953663916 -> 0.00191894953663916

Commit message: Restructured and also exporting to json file for cpp usage

File: 3DOF/urdf/3DOF Yomi Assembly_Anush.urdf (robot description, URDF)
Before this commit: robot 3DOF, 7 links, 6 joints
Links:
- removed link End_effector
Joints:
- removed joint Joint4
